Commit message: ATEMR description model 2

File: urdf/extras/support_macro.urdf.xacro (robot description, xacro)
@@ -11,5 +11,5 @@
         </geometry>
         <xacro:red_material/>
-        <origin xyz="0 0 0" rpy="0 0 ${-pi/2}" />
+        <origin xyz="0 0 0" rpy="0 0 0" />
       </visual>
       <collision>
@@ -18,9 +18,9 @@
         </geometry>
         <xacro:red_material/>
-        <origin xyz="0 0 0" rpy="0 0 ${-pi/2}" />
+        <origin xyz="0 0 0" rpy="0 0 0" />
       </collision>
       <inertial>
         <mass value="${model_mass}" />
-        <origin xyz="0 0 0" rpy="0 0 ${-pi/2}" />
+        <origin xyz="0 0 0" rpy="0 0 0" />
         <inertia  ixx="0.284663364" ixy="-0.000064317" ixz="-0.026604817" iyy="0.285082897" iyz="0.000729986" izz="0.006824376" />
       </inertial>

File: urdf/robot.urdf.xacro (robot description, xacro)
@@ -12,5 +12,5 @@
   <!-- BASE DIMENSIONS -->
   <!-- BASELINK PARAMS -->
-  <xacro:property name="mass" value="3.954"/>
+  <xacro:property name="mass" value="2.79657"/>
   <xacro:property name="base_link_origin">
     <origin rpy="0.0 0.0 0.0" xyz="0.0 -0.002209 0.0405"/>
@@ -18,24 +18,24 @@
   <!-- WHEELS PARAMS -->
   <xacro:property name="has_casters" value="1"/>
-  <xacro:property name="wheel_c_x" value="-0.13589"/>
+  <xacro:property name="wheel_c_x" value="-0.123589"/>
   <xacro:property name="wheel_c_y" value="0.0002"/>
   <xacro:property name="wheel_c_z" value="${-0.00199}"/>
-  <xacro:property name="wheel_l_x" value="0.07283"/>
+  <xacro:property name="wheel_l_x" value="0.060"/>
   <xacro:property name="wheel_l_y" value="0.1589"/>
-  <xacro:property name="wheel_l_z" value="0.026"/>
-  <xacro:property name="wheel_r_x" value="0.07283"/>
+  <xacro:property name="wheel_l_z" value="0.0696"/>
+  <xacro:property name="wheel_r_x" value="0.060"/>
   <xacro:property name="wheel_r_y" value="-0.1589"/>
-  <xacro:property name="wheel_r_z" value="0.026"/>
+  <xacro:property name="wheel_r_z" value="0.0696"/>
   <!-- EXTRAS PARAMS -->
-  <xacro:property name="support_x" value="-0.04478"/>
+  <xacro:property name="support_x" value="-0.08878"/>
   <xacro:property name="support_y" value="0.0"/>
-  <xacro:property name="support_z" value="0.084"/>
+  <xacro:property name="support_z" value="0.11584"/>
   <!-- SENSORS PARAMS -->
-  <xacro:property name="rplidar_x" value="0.00886"/>
-  <xacro:property name="rplidar_y" value="0.00249"/>
-  <xacro:property name="rplidar_z" value="0.169"/>
-  <xacro:property name="rs_cam_x" value="0.12779"/>
-  <xacro:property name="rs_cam_y" value="0.00025"/>
-  <xacro:property name="rs_cam_z" value="0.09029"/>
+  <xacro:property name="rplidar_x" value="-0.00592"/>
+  <xacro:property name="rplidar_y" value="0.0"/>
+  <xacro:property name="rplidar_z" value="0.192"/>
+  <xacro:property name="rs_cam_x" value="0.1093"/>
+  <xacro:property name="rs_cam_y" value="0.00131"/>
+  <xacro:property name="rs_cam_z" value="0.08439"/>
   <!-- ############################ENDCONFIG########################### -->
   <link name="base_footprint"/>
@@ -43,5 +43,5 @@
   <link name="base_link">
     <visual>
-      <origin xyz="0 0 0" rpy="0.0 0.0 ${-pi/2}"/>
+      <origin xyz="0 0 0" rpy="0.0 0.0 0.0"/>
       <geometry>
         <mesh filename="package://atemr_description/meshes/base.dae" scale="1 1 1"/>
@@ -50,5 +50,5 @@
     </visual>
     <collision>
-      <origin xyz="0 0 0" rpy="0.0 0.0 ${-pi/2}"/>
+      <origin xyz="0 0 0" rpy="0.0 0.0 0.0"/>
       <geometry>
         <mesh filename="package://atemr_description/meshes/base_col.stl" scale="1 1 1"/>
@@ -57,6 +57,6 @@
     <inertial>
       <mass value="${mass}" />
-      <origin xyz="0 0 0" rpy="0 0 ${-pi/2}" />
-      <inertia  ixx="0.051523618" ixy="-0.000245748" ixz="0.00165276" iyy="0.060081571" iyz="0.009700999" izz="0.077583265" />
+      <origin xyz="0 0 0" rpy="0 0 0" />
+      <inertia  ixx="0.02493951" ixy="-0.00019788" ixz="-0.000468106" iyy="0.021408522" iyz="0.000079357" izz="0.033811057" />
     </inertial>
   </link>
@@ -81,5 +81,5 @@
   </link>
   <joint name="battery_pack_joint" type="fixed">
-    <origin xyz="-0.04478 0 0.03523" rpy="0 0 0" />
+    <origin xyz="-0.07282 0.0 0.06079" rpy="0 0 0" />
     <parent link="base_link"/>
     <child link="battery_pack"/>

File: urdf/sensors/camera_macro.urdf.xacro (robot description, xacro)
@@ -11,5 +11,5 @@
         </geometry>
         <xacro:red_material/>
-        <origin xyz="0 0 0" rpy="0 0 ${-pi/2}" />
+        <origin xyz="0 0 0" rpy="0 0 0" />
       </visual>
       <collision>
@@ -18,9 +18,9 @@
         </geometry>
         <xacro:red_material/>
-        <origin xyz="0 0 0" rpy="0 0 ${-pi/2}" />
+        <origin xyz="0 0 0" rpy="0 0 0" />
       </collision>
       <inertial>
         <mass value="${model_mass}" />
-        <origin xyz="0 0 0" rpy="0 0 ${-pi/2}" />
+        <origin xyz="0 0 0" rpy="0 0 0" />
         <inertia  ixx="0.000055654" ixy="0.000001199" ixz="-0.000000245" iyy="0.000012386" iyz="-0.000000057" izz="0.000062273" />
       </inertial>
@@ -29,5 +29,5 @@
       <parent link="base_link"/>
       <child link="realsense_camera"/>
-      <origin rpy="0 -0.383972 0" xyz="${x} ${y} ${z}"/>
+      <origin rpy="0 -0.186779 0" xyz="${x} ${y} ${z}"/>
     </joint>
   </xacro:macro>

File: urdf/sensors/irs_macro.urdf.xacro (robot description, xacro)
@@ -9,5 +9,5 @@
       <parent link="base_link"/>
       <child link="irs_front_l"/>
-      <origin rpy="0 0.383972 0" xyz="0 0 0"/>
+      <origin rpy="0 0.383972 0" xyz="0.11406 0.085 0.0"/>
     </joint>
     <link name="irs_front_r" />
@@ -15,5 +15,5 @@
       <parent link="base_link"/>
       <child link="irs_front_r"/>
-      <origin rpy="0 0.383972 0" xyz="0 0 0"/>
+      <origin rpy="0 0.383972 0" xyz="0.11406 -0.085 0.0"/>
     </joint>
     <link name="irs_rear" />
@@ -21,5 +21,5 @@
       <parent link="base_link"/>
       <child link="irs_rear"/>
-      <origin rpy="0 0.383972 0" xyz="0 0 0"/>
+      <origin rpy="0 0.383972 ${pi}" xyz="-0.16006 0.0 0.0"/>
     </joint>
   </xacro:macro>

File: urdf/sensors/rplidar_macro.urdf.xacro (robot description, xacro)
@@ -11,5 +11,5 @@
         </geometry>
         <xacro:red_material/>
-        <origin xyz="0 0 -0.032" rpy="0 0 ${-pi/2}" />
+        <origin xyz="0 0 -0.032" rpy="0 0 0" />
       </visual>
       <collision>
@@ -18,9 +18,9 @@
         </geometry>
         <xacro:red_material/>
-        <origin xyz="0 0 -0.032" rpy="0 0 ${-pi/2}" />
+        <origin xyz="0 0 -0.032" rpy="0 0 0" />
       </collision>
       <inertial>
         <mass value="${model_mass}" />
-        <origin xyz="0 0 -0.032" rpy="0 0 ${-pi/2}" />
+        <origin xyz="0 0 -0.032" rpy="0 0 0" />
         <inertia  ixx="0.000120247" ixy="0.000000595" ixz="0.000002707" iyy="0.000119098" iyz="0.000005916" izz="0.000128464" />
       </inertial>

File: urdf/wheels/caster_wheel_macro.urdf.xacro (robot description, xacro)
@@ -11,5 +11,5 @@
         </geometry>
         <xacro:red_material/>
-        <origin xyz="0 0 0" rpy="0 0 ${pi/2}" />
+        <origin xyz="0 0 0" rpy="0 0 0" />
       </visual>
       <collision>
@@ -18,9 +18,9 @@
         </geometry>
         <xacro:red_material/>
-        <origin xyz="0.02 0 -0.052" rpy="0 0 ${pi/2}" />
+        <origin xyz="0.02 0 -0.052" rpy="0 0 0" />
       </collision>
       <inertial>
         <mass value="${wheel_mass}" />
-        <origin xyz="0 0 0" rpy="0 0 ${pi/2}" />
+        <origin xyz="0 0 0" rpy="0 0 0" />
         <inertia  ixx="0.000102821" ixy="0.000000207" ixz="0.000033294" iyy="0.000117765" iyz="0.00000052" izz="0.000034887" />
       </inertial>

File: urdf/wheels/traction_wheels_macro.urdf.xacro (robot description, xacro)
@@ -14,8 +14,8 @@
         <xacro:red_material/>
         <xacro:if value="${prefix == right_prefix}">
-          <origin xyz="0 0 0" rpy="0 0 ${-pi/2}" />
+          <origin xyz="0 0 0" rpy="${-pi/2} 0 0" />
         </xacro:if>
         <xacro:if value="${prefix == left_prefix}">
-          <origin xyz="0 0 0" rpy="0 0 ${pi/2}" />
+          <origin xyz="0 0 0" rpy="${pi/2} 0 0" />
         </xacro:if>
       </visual>
@@ -26,8 +26,8 @@
         <xacro:red_material/>
         <xacro:if value="${prefix == right_prefix}">
-          <origin xyz="0 0 0" rpy="0 0 ${-pi/2}" />
+          <origin xyz="0 0 0" rpy="${-pi/2} 0 0" />
         </xacro:if>
         <xacro:if value="${prefix == left_prefix}">
-          <origin xyz="0 0 0" rpy="0 0 ${pi/2}" />
+          <origin xyz="0 0 0" rpy="${pi/2} 0 0" />
         </xacro:if>
       </collision>
@@ -35,8 +35,8 @@
         <mass value="${wheel_mass}" />
         <xacro:if value="${prefix == right_prefix}">
-          <origin xyz="0 0 0" rpy="0 0 ${-pi/2}" />
+          <origin xyz="0 0 0" rpy="${-pi/2} 0 0" />
         </xacro:if>
         <xacro:if value="${prefix == left_prefix}">
-          <origin xyz="0 0 0" rpy="0 0 ${pi/2}" />
+          <origin xyz="0 0 0" rpy="${pi/2} 0 0" />
         </xacro:if>
         <inertia  ixx="0.001684091" ixy="0.0" ixz="0.0" iyy="0.001684091" iyz="0.0" izy="0.0" izz="0.0" />
