Commit message: Added new link for 3D camera projection, fixed some simulation parameters

File: urdf/robot.urdf.xacro (robot description, xacro)
@@ -362,5 +362,5 @@
 				<alwaysOn>true</alwaysOn>
 				<updateRate>0.0</updateRate>
-				<cameraName>rs_cam_ir</cameraName>
+				<cameraName>headcamera</cameraName>
 				<imageTopicName>/${robot}/rs_cam/color/image_raw</imageTopicName>
 				<cameraInfoTopicName>/${robot}/rs_cam/color/camera_info</cameraInfoTopicName>
@@ -368,5 +368,5 @@
 				<depthImageCameraInfoTopicName>/${robot}/rs_cam/depth/camera_info</depthImageCameraInfoTopicName>
 				<pointCloudTopicName>/${robot}/rs_cam/depth/points</pointCloudTopicName>
-				<frameName>realsense_camera</frameName>
+				<frameName>realsense_depth_camera</frameName>
 				<pointCloudCutoff>0.5</pointCloudCutoff>
 				<pointCloudCutoffMax>3.0</pointCloudCutoffMax>

File: urdf/sensors/camera_macro.urdf.xacro (robot description, xacro)
@@ -32,4 +32,10 @@
       <origin rpy="0 -0.186779 0" xyz="${x} ${y} ${z}"/>
     </joint>
+    <link name="realsense_depth_camera"/>
+    <joint name="realsense_depth_camera_joint" type="fixed">
+      <parent link="base_link"/>
+      <child link="realsense_depth_camera"/>
+      <origin rpy="${-pi/2 + 0.186779} 0.0 ${-pi/2}" xyz="${x + 0.012} ${y} ${z}"/>
+    </joint>
   </xacro:macro>
 </robot>

Commit message: Prepared real robot launch file

File: urdf/robot.urdf.xacro (robot description, xacro)
@@ -10,5 +10,5 @@
   <xacro:include filename="$(find atemr_description)/urdf/sensors/imu_macro.urdf.xacro"/>
   <!-- Robot properties -->
-  <xacro:property name="robot" value="atemr" />
+  <xacro:property name="robot" value="" />
   <!-- ############################CONFIG########################### -->
   <!-- BASE DIMENSIONS -->
@@ -16,5 +16,5 @@
   <xacro:property name="mass" value="3.0"/>
   <xacro:property name="base_link_origin">
-    <origin rpy="0.0 0.0 0.0" xyz="0.0 -0.002209 0.0405"/>
+    <origin rpy="0.0 0.0 0.0" xyz="-0.060 -0.002209 0.0405"/>
   </xacro:property>
   <!-- WHEELS PARAMS -->
@@ -40,7 +40,7 @@
   <xacro:property name="rs_cam_y" value="0.00131"/>
   <xacro:property name="rs_cam_z" value="0.08439"/>
-  <xacro:property name="imu_x" value="-0.00592"/> <!-- experimental value -->
-  <xacro:property name="imu_y" value="0.0"/> <!-- experimental value -->
-  <xacro:property name="imu_z" value="0.13"/> <!-- experimental value -->
+  <xacro:property name="imu_x" value="${rplidar_x + 0.0257}"/> <!-- experimental value -->
+  <xacro:property name="imu_y" value="${rplidar_y + 0.0065}"/> <!-- experimental value -->
+  <xacro:property name="imu_z" value="0.1115"/> <!-- experimental value -->
   <!-- ############################ENDCONFIG########################### -->
   <link name="base_footprint"/>
@@ -158,6 +158,6 @@
       <wheelSeparation>0.318</wheelSeparation>
       <wheelDiameter>0.108</wheelDiameter>
-      <wheelAcceleration>1.0</wheelAcceleration>
-      <wheelTorque>1.0</wheelTorque>
+      <wheelAcceleration>0.0</wheelAcceleration>
+      <wheelTorque>17</wheelTorque>
       <commandTopic>cmd_vel</commandTopic>
       <odometryTopic>odom</odometryTopic>
@@ -167,5 +167,5 @@
       <publishWheelTF>false</publishWheelTF>
       <publishWheelJointState>true</publishWheelJointState>
-      <publishOdomTF>true</publishOdomTF>
+      <publishOdomTF>false</publishOdomTF>
       <publishTf>true</publishTf>
       <legacyMode>false</legacyMode>

File: urdf/wheels/caster_wheel_macro.urdf.xacro (robot description, xacro)
@@ -3,5 +3,5 @@
   <xacro:include filename="$(find atemr_description)/urdf/common/common.urdf.xacro"/>
   <xacro:include filename="$(find atemr_description)/urdf/common/materials.urdf.xacro"/>
-  <xacro:property name="wheel_mass" value="0.005" />
+  <xacro:property name="wheel_mass" value="0.05" />
   <xacro:macro name="caster_wheel" params="x y z">
     <link name="caster_wheel">

File: urdf/wheels/traction_wheels_macro.urdf.xacro (robot description, xacro)
@@ -5,5 +5,5 @@
   <xacro:property name="right_prefix" value="right" />
   <xacro:property name="left_prefix" value="left" />
-  <xacro:property name="wheel_mass" value="1" />
+  <xacro:property name="wheel_mass" value="0.5" />
   <xacro:macro name="traction_wheel" params="prefix x y z">
     <link name="${prefix}_wheel">

Commit message: Using actual realsense camera description : Re-adjusted IMU sensor position : Re-Adjusted IR sensor angles

File: urdf/robot.urdf.xacro (robot description, xacro)
@@ -6,9 +6,10 @@
   <xacro:include filename="$(find atemr_description)/urdf/extras/support_macro.urdf.xacro"/>
   <xacro:include filename="$(find atemr_description)/urdf/sensors/rplidar_macro.urdf.xacro"/>
-  <xacro:include filename="$(find atemr_description)/urdf/sensors/camera_macro.urdf.xacro"/>
   <xacro:include filename="$(find atemr_description)/urdf/sensors/irs_macro.urdf.xacro"/>
   <xacro:include filename="$(find atemr_description)/urdf/sensors/imu_macro.urdf.xacro"/>
+  <xacro:include filename="$(find realsense2_description)/urdf/_d415.urdf.xacro" />
   <!-- Robot properties -->
   <xacro:property name="robot" value="" />
+  <xacro:property name="camera_name" value="camera" />
   <!-- ############################CONFIG########################### -->
   <!-- BASE DIMENSIONS -->
@@ -37,7 +38,10 @@
   <xacro:property name="rplidar_y" value="0.0"/>
   <xacro:property name="rplidar_z" value="0.192"/>
-  <xacro:property name="rs_cam_x" value="0.1093"/>
+  <xacro:arg name="use_nominal_extrinsics" default="true" />
+  <xacro:arg name="add_plug" default="false" />
+  <xacro:arg name="use_mesh" default="true" />
+  <xacro:property name="rs_cam_x" value="0.1255"/>
   <xacro:property name="rs_cam_y" value="0.00131"/>
-  <xacro:property name="rs_cam_z" value="0.08439"/>
+  <xacro:property name="rs_cam_z" value="0.07310"/>
   <xacro:property name="imu_x" value="${rplidar_x + 0.0257}"/> <!-- experimental value -->
   <xacro:property name="imu_y" value="${rplidar_y + 0.0065}"/> <!-- experimental value -->
@@ -103,5 +107,7 @@
   <!-- SENSORS -->
   <xacro:rplidar x="${rplidar_x}" y="${rplidar_y}" z="${rplidar_z}" />
-  <xacro:realsense_camera x="${rs_cam_x}" y="${rs_cam_y}" z="${rs_cam_z}" />
+  <xacro:sensor_d415 parent="base_link" use_nominal_extrinsics="$(arg use_nominal_extrinsics)" add_plug="$(arg add_plug)" use_mesh="$(arg use_mesh)">
+    <origin xyz="${rs_cam_x} ${rs_cam_y} ${rs_cam_z}" rpy="0.0 -0.3054326 0.0"/> -0.186779
+  </xacro:sensor_d415>
   <xacro:irs />
   <xacro:wt901_imu_sensor x="${imu_x}" y="${imu_y}" z="${imu_z}" />
@@ -150,5 +156,5 @@
   <gazebo>
   	<!--MOTOR CONTROLLER gazebo-->
-    <plugin name="atemr_base_controller" filename="libgazebo_ros_diff_drive.so">
+    <plugin name="base_controller" filename="libgazebo_ros_diff_drive.so">
       <!--robotNamespace>/${robot}</robotNamespace-->
       <updateRate>50</updateRate>
@@ -160,5 +166,5 @@
       <wheelAcceleration>0.0</wheelAcceleration>
       <wheelTorque>17</wheelTorque>
-      <commandTopic>cmd_vel</commandTopic>
+      <commandTopic>base_controller/cmd_vel</commandTopic>
       <odometryTopic>odom</odometryTopic>
       <odometryFrame>odom</odometryFrame>
@@ -310,17 +316,17 @@
 		  <pose>0 0 0 0 0 0</pose>
 			<visualize>false</visualize>
-			<update_rate>10</update_rate>
+			<update_rate>11.5</update_rate>
 			<ray>
 			  <scan>
 				  <horizontal>
-					  <samples>720</samples>
+					  <samples>360</samples>
 						<resolution>0.9</resolution>
-						<min_angle>0.0</min_angle>
-						<max_angle>6.28319</max_angle>
+						<min_angle>0.01745334453880787</min_angle>
+						<max_angle>6.2831854820251465</max_angle>
 					</horizontal>
 				</scan>
 				<range>
-				  <min>0.085</min>
-					<max>6.0</max>
+				  <min>0.15000000596046448</min>
+					<max>12.0</max>
 					<resolution>0.01</resolution>
 				</range>
@@ -332,5 +338,5 @@
 			</ray>
 			<plugin name="gazebo_rplidar_controller" filename="libgazebo_ros_laser.so">
-			  <topicName>/${robot}/laser/scan</topicName>
+			  <topicName>/${robot}/scan</topicName>
 				<frameName>rplidar</frameName>
 			</plugin>
@@ -338,46 +344,46 @@
 	</gazebo>
 	<!--REALENSE CAMERA Sensor gazebo-->
-	<gazebo reference="realsense_camera">
-	  <sensor type="depth" name="rs_cam">
+	<gazebo reference="camera_bottom_screw_frame"> <!-- link name-->
+	  <sensor name="d415_camera" type="depth">
 		  <update_rate>20.0</update_rate>
-			<camera name="headcamera">
-			  <!--horizontal_fov>1.22173</horizontal_fov-->
+			<camera>
+			  <horizontal_fov>1.204280</horizontal_fov>
 				<image>
-				  <width>480</width>
-					<height>270</height>
+				  <width>640</width>
+					<height>480</height>
 					<format>R8G8B8</format>
 				</image>
 				<clip>
 				  <near>0.05</near>
-					<far>30</far>
+					<far>3</far>
 				</clip>
 				<noise>
 				  <type>gaussian</type>
 					<mean>0.0</mean>
-					<stddev>0.003</stddev>
+					<stddev>0.0003</stddev>
 				</noise>
 			</camera>
-			<plugin name="kinect" filename="libgazebo_ros_openni_kinect.so">
+			<plugin name="d415_camera_controller" filename="libgazebo_ros_openni_kinect.so">
 			  <baseline>0.055</baseline>
 				<alwaysOn>true</alwaysOn>
-				<updateRate>0.0</updateRate>
-				<cameraName>headcamera</cameraName>
-				<imageTopicName>/${robot}/rs_cam/color/image_raw</imageTopicName>
-				<cameraInfoTopicName>/${robot}/rs_cam/color/camera_info</cameraInfoTopicName>
-				<depthImageTopicName>/${robot}/rs_cam/depth/image_raw</depthImageTopicName>
-				<depthImageCameraInfoTopicName>/${robot}/rs_cam/depth/camera_info</depthImageCameraInfoTopicName>
-				<pointCloudTopicName>/${robot}/rs_cam/depth/points</pointCloudTopicName>
-				<frameName>realsense_depth_camera</frameName>
+				<updateRate>1.0</updateRate>
+				<cameraName>${camera_name}_ir</cameraName>
+				<imageTopicName>/${robot}/${camera_name}/color/image_raw</imageTopicName>
+				<cameraInfoTopicName>/${robot}/${camera_name}/color/camera_info</cameraInfoTopicName>
+				<depthImageTopicName>/${robot}/${camera_name}/depth/image_raw</depthImageTopicName>
+				<depthImageCameraInfoTopicName>/${robot}/${camera_name}/depth/camera_info</depthImageCameraInfoTopicName>
+				<pointCloudTopicName>/${robot}/${camera_name}/depth/points</pointCloudTopicName>
+				<frameName>camera_depth_optical_frame</frameName>
 				<pointCloudCutoff>0.5</pointCloudCutoff>
 				<pointCloudCutoffMax>3.0</pointCloudCutoffMax>
-				<distortionK1>0</distortionK1>
-				<distortionK2>0</distortionK2>
-				<distortionK3>0</distortionK3>
-				<distortionT1>0</distortionT1>
-				<distortionT2>0</distortionT2>
+				<distortionK1>0.00000001</distortionK1>
+				<distortionK2>0.00000001</distortionK2>
+				<distortionK3>0.00000001</distortionK3>
+				<distortionT1>0.00000001</distortionT1>
+				<distortionT2>0.00000001</distortionT2>
 				<CxPrime>0</CxPrime>
 				<Cx>0</Cx>
 				<Cy>0</Cy>
-				<!--focalLength>0.00188</focalLength-->
+				<focalLength>465.601485</focalLength> <!-- 0.0 -->
 				<hackBaseline>0</hackBaseline>
 			</plugin>

File: urdf/sensors/camera_macro.urdf.xacro (robot description, xacro)
@@ -5,5 +5,5 @@
   <xacro:property name="model_mass" value="0.072" />
   <xacro:macro name="realsense_camera" params="x y z">
-    <link name="realsense_camera">
+    <link name="rs_camera_link">
       <visual>
         <geometry>
@@ -27,13 +27,13 @@
       </inertial>
     </link>
-    <joint name="realsense_camera_joint" type="fixed">
+    <joint name="rs_camera_joint" type="fixed">
       <parent link="base_link"/>
-      <child link="realsense_camera"/>
+      <child link="rs_camera_link"/>
       <origin rpy="0 -0.186779 0" xyz="${x} ${y} ${z}"/>
     </joint>
-    <link name="realsense_depth_camera"/>
-    <joint name="realsense_depth_camera_joint" type="fixed">
+    <link name="rs_depth_camera"/>
+    <joint name="rs_depth_camera_joint" type="fixed">
       <parent link="base_link"/>
-      <child link="realsense_depth_camera"/>
+      <child link="rs_depth_camera"/>
       <origin rpy="${-pi/2 + 0.186779} 0.0 ${-pi/2}" xyz="${x + 0.012} ${y} ${z}"/>
     </joint>

File: urdf/sensors/irs_macro.urdf.xacro (robot description, xacro)
@@ -9,5 +9,5 @@
       <parent link="base_link"/>
       <child link="irs_front_l"/>
-      <origin rpy="0 0.383972 0" xyz="0.11406 0.085 0.0"/>
+      <origin rpy="0 0.29670 0" xyz="0.11406 0.085 0.0"/>
     </joint>
     <link name="irs_front_r" />
@@ -15,5 +15,5 @@
       <parent link="base_link"/>
       <child link="irs_front_r"/>
-      <origin rpy="0 0.383972 0" xyz="0.11406 -0.085 0.0"/>
+      <origin rpy="0 0.29670 0" xyz="0.11406 -0.085 0.0"/>
     </joint>
     <link name="irs_rear" />
@@ -21,5 +21,5 @@
       <parent link="base_link"/>
       <child link="irs_rear"/>
-      <origin rpy="0 0.383972 ${pi}" xyz="-0.16006 0.0 0.0"/>
+      <origin rpy="0 0.29670 ${pi}" xyz="-0.16006 0.0 0.0"/>
     </joint>
   </xacro:macro>
