Commit message: Fixed IMU orientation

File: urdf/sensors/imu_macro.urdf.xacro (robot description, xacro)
@@ -3,5 +3,5 @@
   <xacro:include filename="$(find atemr_description)/urdf/common/common.urdf.xacro"/>
   <xacro:include filename="$(find atemr_description)/urdf/common/materials.urdf.xacro"/>
-  <xacro:property name="model_mass" value="0.050" />
+  <xacro:property name="model_mass" value="0.010" />
   <xacro:macro name="wt901_imu_sensor" params="x y z">
     <link name="wt901_imu" />
@@ -9,5 +9,5 @@
       <parent link="base_link"/>
       <child link="wt901_imu"/>
-      <origin rpy="0 0 0" xyz="${x} ${y} ${z}"/>
+      <origin rpy="0 0 ${-pi/2}" xyz="${x} ${y} ${z}"/>
     </joint>
   </xacro:macro>

Commit message: Fixed IMU URDF

File: urdf/sensors/imu_macro.urdf.xacro (robot description, xacro)
@@ -9,5 +9,5 @@
       <parent link="base_link"/>
       <child link="wt901_imu"/>
-      <origin rpy="0 0 ${-pi/2}" xyz="${x} ${y} ${z}"/>
+      <origin rpy="0 0 0" xyz="${x} ${y} ${z}"/>
     </joint>
   </xacro:macro>
